File: osw-light.sch (KiCad schematic (older format))
At the start: 65 parts, among them J1 Conn_01x02, Q1 2N7002, SW1 SW_Push, SW2 SW_Push, SW4 SW_Push, SW5 SW_Push, U1 DS3231MZ, U10 XC6209, U11 MCP73831T-2ACI_OT, U12 USBLC6-2SC6, U13 XC6209, U2 BMA400, U3 BMP280, U4 GC9A01_IPS_display, U5 USB-OTG, U6 CH340E, U7 ttgo-32-micro, U8 Quectel_L96, U9 TPS2115A

Commit message: osw light v1.0
Parts:
- removed C10, C7: 0.1u, Capacitor_SMD:C_0603_1608Metric, symbol Device:C_Small
- removed C20: 100p, Capacitor_SMD:C_0603_1608Metric, symbol Device:C_Small
- removed C21: 10p, Capacitor_SMD:C_0603_1608Metric, symbol Device:C_Small
- removed R12: 5.6k, Resistor_SMD:R_0603_1608Metric, symbol Device:R_Small
- removed R2, R3: 1k, Resistor_SMD:R_0603_1608Metric, symbol Device:R_Small
- removed R5: 0R, Resistor_SMD:R_0402_1005Metric, symbol Device:R_Small
- removed U8: Quectel_L96, open-Smartwatch:Quectel_L96, symbol open-Smartwatch:Quectel_L96
- removed XS1: SD_ebay-uSD-push_push_SMD, open-Smartwatch:Conn_uSDcard, symbol open-Smartwatch:SD_ebay-uSD-push_push_SMD
Connections:
- net GPS_RX3V3: no longer names the net of U7.13 (IO14)
- net GPS_TX3V3: no longer names the net of U7.12 (IO27)
- net MISO: no longer names the net of U7.31 (IO19)
- net SD_CS: no longer names the net of U7.26 (IO04)
- no-connect marks 30 -> 21
Other:
- note removed: "0 Ohm across\nRFin/RFout for\ninternal antenna"
- note removed: "GPS"
- note removed: "SDCARD"
